File: building_blocks.kicad_sch (KiCad schematic)
At the start: 50 parts, among them J1 conn_1x3, J10 conn_1x3, J2 conn_1x3, J3 conn_1x3, J5 conn_1x3, J6 conn_1x3, J7 conn_1x3, J8 conn_1x3, J9 conn_1x3, Q1 LBSS84LT1G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

Commit message: Added kikit fab script
Parts:
- Q1, Q2, Q3, Q4: JLCPCB_CORRECTION 0;0;0 -> 0;0;180
- R8: value 91k 0.1% -> 180k 0.1%
- R9: value 10k 1% -> 20k; LCSC C25744 -> C25765
- U1, U2, U3, U4: JLCPCB_CORRECTION (none) -> 0;0;270
Changed lines of the file:
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@@
+      (effects (font (size 1.27 1.27)) hide)
+    )
+    (property "JLCPCB_CORRECTION" "0;0;270" (id 5) (at 124.46 70.485 0)
       (effects (font (size 1.27 1.27)) hide)
     )
@@
       (effects (font (size 1.27 1.27)) hide)
     )
-    (property "JLCPCB_CORRECTION" "0;0;0" (id 5) (at 231.14 219.71 90)
+    (property "JLCPCB_CORRECTION" "0;0;180" (id 5) (at 231.14 219.71 90)
       (effects (font (size 1.27 1.27)) hide)
     )
@@
     )
     (property "LCSC" "C1850244" (id 4) (at 124.46 180.34 0)
+      (effects (font (size 1.27 1.27)) hide)
+    )
+    (property "JLCPCB_CORRECTION" "0;0;270" (id 5) (at 124.46 180.34 0)
       (effects (font (size 1.27 1.27)) hide)
     )
@@
     (in_bom yes) (on_board yes)
     (property "Reference" "R8" (id 0) (at 141.605 193.04 90))
-    (property "Value" "91k 0.1%" (id 1) (at 139.7 191.77 90))
+    (property "Value" "180k 0.1%" (id 1) (at 139.7 191.77 90))
     (property "Footprint" "Resistor_SMD:R_0603_1608Metric" (id 2) (at 134.747 190.5 90)
       (effects (font (size 1.27 1.27)) hide)
@@
     )
     (property "LCSC" "C1850244" (id 4) (at 267.335 71.755 0)
+      (effects (font (size 1.27 1.27)) hide)
+    )
+    (property "JLCPCB_CORRECTION" "0;0;270" (id 5) (at 267.335 71.755 0)
       (effects (font (size 1.27 1.27)) hide)
     )
@@
     (in_bom yes) (on_board yes)
     (property "Reference" "R9" (id 0) (at 139.7 212.09 90))
-    (property "Value" "10k 1%" (id 1) (at 141.605 211.455 90))
+    (property "Value" "20k" (id 1) (at 141.605 211.455 90))
     (property "Footprint" "Resistor_SMD:R_0402_1005Metric" (id 2) (at 138.303 209.55 90)
       (effects (font (size 1.27 1.27)) hide)
@@
       (effects (font (size 1.27 1.27)) hide)
     )
-    (property "LCSC" "C25744" (id 4) (at 136.525 209.55 0)
+    (property "LCSC" "C25765" (id 4) (at 136.525 209.55 0)
       (effects (font (size 1.27 1.27)) hide)
     )
@@
       (effects (font (size 1.27 1.27)) hide)
     )
-    (property "JLCPCB_CORRECTION" "0;0;0" (id 5) (at 63.5 219.075 90)
+    (property "JLCPCB_CORRECTION" "0;0;180" (id 5) (at 63.5 219.075 90)
       (effects (font (size 1.27 1.27)) hide)
     )
@@
       (effects (font (size 1.27 1.27)) hide)
     )
-    (property "JLCPCB_CORRECTION" "0;0;0" (id 5) (at 231.14 109.855 90)
+    (property "JLCPCB_CORRECTION" "0;0;180" (id 5) (at 231.14 109.855 90)
       (effects (font (size 1.27 1.27)) hide)
     )
@@
       (effects (font (size 1.27 1.27)) hide)
     )
-    (property "JLCPCB_CORRECTION" "0;0;0" (id 5) (at 71.12 109.855 90)
+    (property "JLCPCB_CORRECTION" "0;0;180" (id 5) (at 71.12 109.855 90)
       (effects (font (size 1.27 1.27)) hide)
     )
@@
       (effects (font (size 1.27 1.27)) hide)
     )
+    (property "JLCPCB_CORRECTION" "0;0;270" (id 5) (at 259.715 183.515 0)
+      (effects (font (size 1.27 1.27)) hide)
+    )
     (pin "2")
     (pin "5")
@@
     )
     (path "/361a6aa7-9206-4064-b3c2-eb1e95593124"
-      (reference "R8") (unit 1) (value "91k 0.1%") (footprint "Resistor_SMD:R_0603_1608Metric")
+      (reference "R8") (unit 1) (value "180k 0.1%") (footprint "Resistor_SMD:R_0603_1608Metric")
     )
     (path "/4922e12c-87b7-4df0-9c25-95ca579a53e8"
-      (reference "R9") (unit 1) (value "10k 1%") (footprint "Resistor_SMD:R_0402_1005Metric")
+      (reference "R9") (unit 1) (value "20k") (footprint "Resistor_SMD:R_0402_1005Metric")
     )
     (path "/40029999-58fe-494c-b419-d488a7cd4322"
